File: modules/SENSOR.kicad_sch (KiCad schematic)
At the start: 7 parts, among them Q2 AO3400A, U12 BME280

Commit message: save
Parts:
- Q2: footprint Package_TO_SOT_SMD:TSOT-23 -> Package_TO_SOT_SMD:SOT-23; symbol Device:Q_NMOS -> Transistor_FET:Q_NMOS_DGS
Connections:
- net GND: now also Q2.3 (S); no longer Q2.S
- net PWM_BUZZER: now also Q2.2 (G); no longer Q2.G
- net at BZ1.2 (-), D2.2 (A): now also Q2.1 (D); no longer Q2.D
Changed lines of the file:
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@@
 	)
 	(symbol
-		(lib_id "Device:Q_NMOS")
+		(lib_id "Transistor_FET:Q_NMOS_DGS")
 		(at 187.96 102.87 0)
 		(unit 1)
@@
 			)
 		)
-		(property "Footprint" "Package_TO_SOT_SMD:TSOT-23"
+		(property "Footprint" "Package_TO_SOT_SMD:SOT-23"
 			(at 193.04 100.33 0)
 			(effects
@@
 			)
 		)
-		(property "Datasheet" "https://mm.digikey.com/Volume0/opasdata/d220001/medias/docus/1133/AO3400A_ds.pdf"
+		(property "Datasheet" "~"
 			(at 187.96 102.87 0)
 			(effects
@@
 			)
 		)
-		(property "Description" "N-Channel 30 V 5.7A (Ta) 1.4W (Ta) Surface Mount SOT-23-3"
+		(property "Description" "N-MOSFET transistor, drain/gate/source"
 			(at 187.96 102.87 0)
 			(effects
@@
 			)
 		)
-		(pin "S"
+		(pin "1"
 		)
-		(pin "G"
+		(pin "2"
 		)
-		(pin "D"
+		(pin "3"
 		)
 		(instances

Commit message: Cambio de layout, correccion de pinout
Parts:
- renumbered U12 to U6
Changed lines of the file:
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@@
 		(instances
 			(project "RP_devBoard"
-				(path "/3efb3214-cf20-4475-a403-c426a77bfef6/c6764cad-48c1-4f00-be75-4674e72510ab"
+				(path "/3efb3214-cf20-4475-a403-c426a77bfef6/62113720-2c63-473f-95b5-ca8de1b9712b"
 					(reference "C33")
 					(unit 1)
@@
 		(instances
 			(project "RP_devBoard"
-				(path "/3efb3214-cf20-4475-a403-c426a77bfef6/c6764cad-48c1-4f00-be75-4674e72510ab"
+				(path "/3efb3214-cf20-4475-a403-c426a77bfef6/62113720-2c63-473f-95b5-ca8de1b9712b"
 					(reference "R22")
 					(unit 1)
@@
 		)
 		(instances
-			(project ""
-				(path "/3efb3214-cf20-4475-a403-c426a77bfef6/c6764cad-48c1-4f00-be75-4674e72510ab"
+			(project "RP_devBoard"
+				(path "/3efb3214-cf20-4475-a403-c426a77bfef6/62113720-2c63-473f-95b5-ca8de1b9712b"
 					(reference "D2")
 					(unit 1)
@@
 		(on_board yes)
 		(dnp no)
-		(property "Reference" "#PWR054"
+		(property "Reference" "#PWR033"
 			(at 80.01 123.19 0)
 			(effects
@@
 		(instances
 			(project "RP_devBoard"
-				(path "/3efb3214-cf20-4475-a403-c426a77bfef6/c6764cad-48c1-4f00-be75-4674e72510ab"
-					(reference "#PWR054")
+				(path "/3efb3214-cf20-4475-a403-c426a77bfef6/62113720-2c63-473f-95b5-ca8de1b9712b"
+					(reference "#PWR033")
 					(unit 1)
 				)
@@
 		(on_board yes)
 		(dnp no)
-		(property "Reference" "#PWR055"
+		(property "Reference" "#PWR050"
 			(at 85.09 123.19 0)
 			(effects
@@
 		(instances
 			(project "RP_devBoard"
-				(path "/3efb3214-cf20-4475-a403-c426a77bfef6/c6764cad-48c1-4f00-be75-4674e72510ab"
-					(reference "#PWR055")
+				(path "/3efb3214-cf20-4475-a403-c426a77bfef6/62113720-2c63-473f-95b5-ca8de1b9712b"
+					(reference "#PWR050")
 					(unit 1)
 				)
@@
 		)
 		(instances
-			(project ""
-				(path "/3efb3214-cf20-4475-a403-c426a77bfef6/c6764cad-48c1-4f00-be75-4674e72510ab"
+			(project "RP_devBoard"
+				(path "/3efb3214-cf20-4475-a403-c426a77bfef6/62113720-2c63-473f-95b5-ca8de1b9712b"
 					(reference "Q2")
 					(unit 1)
@@
 		(on_board yes)
 		(dnp no)
-		(property "Reference" "#PWR032"
+		(property "Reference" "#PWR055"
 			(at 190.5 121.92 0)
 			(effects
@@
 		(instances
 			(project "RP_devBoard"
-				(path "/3efb3214-cf20-4475-a403-c426a77bfef6/c6764cad-48c1-4f00-be75-4674e72510ab"
-					(reference "#PWR032")
+				(path "/3efb3214-cf20-4475-a403-c426a77bfef6/62113720-2c63-473f-95b5-ca8de1b9712b"
+					(reference "#PWR055")
 					(unit 1)
 				)
@@
 		(instances
 			(project "RP_devBoard"
-				(path "/3efb3214-cf20-4475-a403-c426a77bfef6/c6764cad-48c1-4f00-be75-4674e72510ab"
+				(path "/3efb3214-cf20-4475-a403-c426a77bfef6/62113720-2c63-473f-95b5-ca8de1b9712b"
 					(reference "C34")
 					(unit 1)
@@
 		)
 		(instances
-			(project ""
-				(path "/3efb3214-cf20-4475-a403-c426a77bfef6/c6764cad-48c1-4f00-be75-4674e72510ab"
+			(project "RP_devBoard"
+				(path "/3efb3214-cf20-4475-a403-c426a77bfef6/62113720-2c63-473f-95b5-ca8de1b9712b"
 					(reference "BZ1")
 					(unit 1)
@@
 		(dnp no)
 		(fields_autoplaced yes)
-		(property "Reference" "U12"
+		(property "Reference" "U6"
 			(at 71.12 97.7899 0)
 			(effects
@@
 		(instances
 			(project "RP_devBoard"
-				(path "/3efb3214-cf20-4475-a403-c426a77bfef6/c6764cad-48c1-4f00-be75-4674e72510ab"
-					(reference "U12")
+				(path "/3efb3214-cf20-4475-a403-c426a77bfef6/62113720-2c63-473f-95b5-ca8de1b9712b"
+					(reference "U6")
 					(unit 1)
 				)
@@
 		(on_board yes)
 		(dnp no)
-		(property "Reference" "#PWR033"
+		(property "Reference" "#PWR054"
 			(at 175.26 121.92 0)
 			(effects
@@
 		(instances
 			(project "RP_devBoard"
-				(path "/3efb3214-cf20-4475-a403-c426a77bfef6/c6764cad-48c1-4f00-be75-4674e72510ab"
-					(reference "#PWR033")
+				(path "/3efb3214-cf20-4475-a403-c426a77bfef6/62113720-2c63-473f-95b5-ca8de1b9712b"
+					(reference "#PWR054")
 					(unit 1)
 				)
@@
 		(on_board yes)
 		(dnp no)
-		(property "Reference" "#PWR050"
+		(property "Reference" "#PWR032"
 			(at 67.31 87.63 0)
 			(effects
@@
 		(instances
 			(project "RP_devBoard"
-				(path "/3efb3214-cf20-4475-a403-c426a77bfef6/c6764cad-48c1-4f00-be75-4674e72510ab"
-					(reference "#PWR050")
+				(path "/3efb3214-cf20-4475-a403-c426a77bfef6/62113720-2c63-473f-95b5-ca8de1b9712b"
+					(reference "#PWR032")
 					(unit 1)
 				)
@@
 		(instances
 			(project "RP_devBoard"
-				(path "/3efb3214-cf20-4475-a403-c426a77bfef6/c6764cad-48c1-4f00-be75-4674e72510ab"
+				(path "/3efb3214-cf20-4475-a403-c426a77bfef6/62113720-2c63-473f-95b5-ca8de1b9712b"
 					(reference "#PWR051")
 					(unit 1)
