File: modules/RP2350B.kicad_sch (KiCad schematic)
At the start: 49 parts, among them SW1 SW_Push, SW3 SW_Push, SW4 SW_Push, U1 RP2350B, U5 W25Q128JVS, Y1 12MHz

Commit message: finishing version 1.0
Parts:
- C16, C18, C38, C9: Part Number CL05B104KA5NNNC -> C0603C104K5RACTU
- C4, C8: Part Number GRM155D71A475ME15J -> GRM188R61E475KE11D
- R18, R6: Part Number ERJ-2RKF1001X -> RMCF0603FT1K00
- R20: footprint Capacitor_SMD:C_0603_1608Metric -> Resistor_SMD:R_0603_1608Metric; Part Number ERJ-2RKF1001X -> RMCF0603FT1K00
Connections:
- no-connect marks 1 -> 23
Changed lines of the file:
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@@
 	)
 	(junction
+		(at 22.86 80.01)
+		(diameter 0)
+		(color 0 0 0 0)
+	)
+	(junction
 		(at 38.1 21.59)
 		(diameter 0)
@@
 	)
 	(no_connect
+		(at 124.46 87.63)
+	)
+	(no_connect
+		(at 124.46 120.65)
+	)
+	(no_connect
+		(at 124.46 110.49)
+	)
+	(no_connect
+		(at 124.46 82.55)
+	)
+	(no_connect
+		(at 124.46 90.17)
+	)
+	(no_connect
+		(at 124.46 92.71)
+	)
+	(no_connect
+		(at 124.46 167.64)
+	)
+	(no_connect
 		(at 124.46 69.85)
 	)
+	(no_connect
+		(at 124.46 118.11)
+	)
+	(no_connect
+		(at 124.46 107.95)
+	)
+	(no_connect
+		(at 124.46 128.27)
+	)
+	(no_connect
+		(at 124.46 95.25)
+	)
+	(no_connect
+		(at 124.46 80.01)
+	)
+	(no_connect
+		(at 124.46 85.09)
+	)
+	(no_connect
+		(at 124.46 115.57)
+	)
+	(no_connect
+		(at 124.46 130.81)
+	)
+	(no_connect
+		(at 124.46 125.73)
+	)
+	(no_connect
+		(at 124.46 158.75)
+	)
+	(no_connect
+		(at 124.46 77.47)
+	)
+	(no_connect
+		(at 124.46 123.19)
+	)
+	(no_connect
+		(at 124.46 102.87)
+	)
+	(no_connect
+		(at 124.46 113.03)
+	)
+	(no_connect
+		(at 124.46 105.41)
+	)
 	(bus_entry
 		(at 58.42 91.44)
@@
 	(wire
 		(pts
+			(xy 22.86 68.58) (xy 22.86 80.01)
+		)
+		(stroke
+			(width 0)
+			(type default)
+		)
+	)
+	(wire
+		(pts
 			(xy 119.38 31.75) (xy 132.08 31.75)
 		)
@@
 	(wire
 		(pts
-			(xy 20.32 80.01) (xy 26.67 80.01)
+			(xy 20.32 80.01) (xy 22.86 80.01)
 		)
 		(stroke
@@
 	(wire
 		(pts
-			(xy 124.46 158.75) (xy 133.35 158.75)
-		)
-		(stroke
-			(width 0)
-			(type default)
-		)
-	)
-	(wire
-		(pts
 			(xy 30.48 115.57) (xy 38.1 115.57)
 		)
@@
 	(wire
 		(pts
-			(xy 161.29 171.45) (xy 166.37 171.45)
-		)
-		(stroke
-			(width 0)
-			(type default)
-		)
-	)
-	(wire
-		(pts
 			(xy 223.52 48.26) (xy 229.87 48.26)
 		)
@@
 	(wire
 		(pts
-			(xy 133.35 167.64) (xy 124.46 167.64)
-		)
-		(stroke
-			(width 0)
-			(type default)
-		)
-	)
-	(wire
-		(pts
 			(xy 245.11 99.06) (xy 245.11 106.68)
 		)
@@
 	(wire
 		(pts
-			(xy 161.29 173.99) (xy 166.37 173.99)
+			(xy 22.86 80.01) (xy 26.67 80.01)
 		)
 		(stroke
@@
 		)
 	)
-	(hierarchical_label "RPB_SWO"
-		(shape output)
-		(at 166.37 171.45 0)
-		(effects
-			(font
-				(size 1.27 1.27)
-			)
-			(justify left)
-		)
-	)
 	(hierarchical_label "USB_DN"
 		(shape bidirectional)
@@
 			)
 		)
-		(property "Datasheet" "https://mm.digikey.com/Volume0/opasdata/d220001/medias/docus/729/CL05B104KA5NNNC_Spec.pdf"
+		(property "Datasheet" "https://yageogroup.com/content/datasheet/asset/file/KEM_C1002_X7R_SMD"
 			(at 36.83 163.83 0)
 			(effects
@@
 			)
 		)
-		(property "Description" "CAP CER 0.1UF 25V X7R 0402"
+		(property "Description" "CAP CER 0.1UF 50V X7R 0603"
 			(at 36.83 163.83 0)
 			(effects
@@
 			)
 		)
-		(property "Part Number" "CL05B104KA5NNNC"
+		(property "Part Number" "C0603C104K5RACTU"
 			(at 36.83 163.83 0)
 			(effects
@@
 			)
 		)
-		(property "Datasheet" "https://industrial.panasonic.com/cdbs/www-data/pdf/RDA0000/AOA0000C304.pdf"
+		(property "Datasheet" "https://www.seielect.com/catalog/SEI-RMCF_RMCP.pdf"
 			(at 167.64 121.92 0)
 			(effects
@@
 			)
 		)
-		(property "Description" "RES SMD 1K OHM 1% 1/10W 0402"
+		(property "Description" "RES 1K OHM 1% 1/10W 0603"
 			(at 167.64 121.92 0)
 			(effects
@@
 			)
 		)
-		(property "Part Number" "ERJ-2RKF1001X"
+		(property "Part Number" "RMCF0603FT1K00"
 			(at 167.64 121.92 90)
 			(effects
@@
 			)
 		)
-		(property "Datasheet" "https://search.murata.co.jp/Ceramy/image/img/A01X/G101/ENG/GRM155D71A475ME15-01A.pdf"
+		(property "Datasheet" "https://search.murata.co.jp/Ceramy/image/img/A01X/G101/ENG/GRM188R61E475KE11-01.pdf"
 			(at 20.32 86.36 0)
 			(effects
@@
 			)
 		)
-		(property "Description" "CAP CER 4.7UF 10V X7T 0402"
+		(property "Description" "CAP CER 4.7UF 25V X5R 0603"
 			(at 20.32 86.36 0)
 			(effects
@@
 			)
 		)
-		(property "Part Number" "GRM155D71A475ME15J"
+		(property "Part Number" "GRM188R61E475KE11D"
 			(at 20.32 86.36 0)
 			(effects
@@
 			)
 		)
-		(property "Datasheet" "https://mm.digikey.com/Volume0/opasdata/d220001/medias/docus/729/CL05B104KA5NNNC_Spec.pdf"
+		(property "Datasheet" "https://yageogroup.com/content/datasheet/asset/file/KEM_C1002_X7R_SMD"
 			(at 240.03 52.07 0)
 			(effects
@@
 			)
 		)
-		(property "Description" "CAP CER 0.1UF 25V X7R 0402"
+		(property "Description" "CAP CER 0.1UF 50V X7R 0603"
 			(at 240.03 52.07 0)
 			(effects
@@
 			)
 		)
-		(property "Part Number" "CL05B104KA5NNNC"
+		(property "Part Number" "C0603C104K5RACTU"
 			(at 240.03 52.07 0)
 			(effects
@@
 			)
 		)
-		(property "Datasheet" "https://mm.digikey.com/Volume0/opasdata/d220001/medias/docus/729/CL05B104KA5NNNC_Spec.pdf"
+		(property "Datasheet" "https://yageogroup.com/content/datasheet/asset/file/KEM_C1002_X7R_SMD"
 			(at 140.97 96.52 0)
 			(effects
@@
 			)
 		)
-		(property "Description" "CAP CER 0.1UF 25V X7R 0402"
+		(property "Description" "CAP CER 0.1UF 50V X7R 0603"
 			(at 140.97 96.52 0)
 			(effects
@@
 			)
 		)
-		(property "Part Number" "CL05B104KA5NNNC"
+		(property "Part Number" "C0603C104K5RACTU"
 			(at 140.97 96.52 0)
 			(effects
@@
 			)
 		)
-		(property "Datasheet" "https://search.murata.co.jp/Ceramy/image/img/A01X/G101/ENG/GRM155D71A475ME15-01A.pdf"
+		(property "Datasheet" "https://search.murata.co.jp/Ceramy/image/img/A01X/G101/ENG/GRM188R61E475KE11-01.pdf"
 			(at 46.99 54.61 0)
 			(effects
@@
 			)
 		)
-		(property "Description" "CAP CER 4.7UF 10V X7T 0402"
+		(property "Description" "CAP CER 4.7UF 25V X5R 0603"
 			(at 46.99 54.61 0)
 			(effects
@@
 			)
 		)
-		(property "Part Number" "GRM155D71A475ME15J"
+		(property "Part Number" "GRM188R61E475KE11D"
 			(at 46.99 54.61 0)
 			(effects
@@
 	)
 	(symbol
+		(lib_id "power:PWR_FLAG")
+		(at 22.86 68.58 0)
+		(unit 1)
+		(exclude_from_sim no)
+		(in_bom yes)
+		(on_board yes)
+		(dnp no)
+		(fields_autoplaced yes)
+		(property "Reference" "#FLG08"
+			(at 22.86 66.675 0)
+			(effects
+				(font
+					(size 1.27 1.27)
+				)
+				(hide yes)
+			)
+		)
+		(property "Value" "PWR_FLAG"
+			(at 22.86 63.5 0)
+			(effects
+				(font
+					(size 1.27 1.27)
+				)
+			)
+		)
+		(property "Footprint" ""
+			(at 22.86 68.58 0)
+			(effects
+				(font
+					(size 1.27 1.27)
+				)
+				(hide yes)
+			)
+		)
+		(property "Datasheet" "~"
+			(at 22.86 68.58 0)
+			(effects
+				(font
+					(size 1.27 1.27)
+				)
+				(hide yes)
+			)
+		)
+		(property "Description" "Special symbol for telling ERC where power comes from"
+			(at 22.86 68.58 0)
+			(effects
+				(font
+					(size 1.27 1.27)
+				)
+				(hide yes)
+			)
+		)
+		(pin "1"
+		)
+		(instances
+			(project "RP_devBoard"
+				(path "/3efb3214-cf20-4475-a403-c426a77bfef6/a6247f93-6950-41b7-9157-645e57be43d7"
+					(reference "#FLG08")
+					(unit 1)
+				)
+			)
+		)
+	)
+	(symbol
 		(lib_id "Device:C")
 		(at 50.8 26.67 0)
@@
 			)
 		)
-		(property "Datasheet" "https://industrial.panasonic.com/cdbs/www-data/pdf/RDA0000/AOA0000C304.pdf"
+		(property "Datasheet" "https://www.seielect.com/catalog/SEI-RMCF_RMCP.pdf"
 			(at 45.72 179.07 0)
 			(effects
@@
 			)
 		)
-		(property "Description" "RES SMD 1K OHM 1% 1/10W 0402"
+		(property "Description" "RES 1K OHM 1% 1/10W 0603"
 			(at 45.72 179.07 0)
 			(effects
@@
 			)
 		)
-		(property "Part Number" "ERJ-2RKF1001X"
+		(property "Part Number" "RMCF0603FT1K00"
 			(at 45.72 179.07 90)
 			(effects
@@
 			)
 		)
-		(property "Datasheet" "https://mm.digikey.com/Volume0/opasdata/d220001/medias/docus/729/CL05B104KA5NNNC_Spec.pdf"
+		(property "Datasheet" "https://yageogroup.com/content/datasheet/asset/file/KEM_C1002_X7R_SMD"
 			(at 163.83 99.06 0)
 			(effects
@@
 			)
 		)
-		(property "Description" "CAP CER 0.1UF 25V X7R 0402"
+		(property "Description" "CAP CER 0.1UF 50V X7R 0603"
 			(at 163.83 99.06 0)
 			(effects
@@
 			)
 		)
-		(property "Part Number" "CL05B104KA5NNNC"
+		(property "Part Number" "C0603C104K5RACTU"
 			(at 163.83 99.06 0)
 			(effects
@@
 			)
 		)
-		(property "Footprint" "Capacitor_SMD:C_0603_1608Metric"
+		(property "Footprint" "Resistor_SMD:R_0603_1608Metric"
 			(at 200.66 116.332 90)
 			(effects
@@
 			)
 		)
-		(property "Datasheet" "https://industrial.panasonic.com/cdbs/www-data/pdf/RDA0000/AOA0000C304.pdf"
+		(property "Datasheet" "https://www.seielect.com/catalog/SEI-RMCF_RMCP.pdf"
 			(at 200.66 118.11 0)
 			(effects
@@
 			)
 		)
-		(property "Description" "RES SMD 1K OHM 1% 1/10W 0402"
+		(property "Description" "RES 1K OHM 1% 1/10W 0603"
 			(at 200.66 118.11 0)
 			(effects
@@
 			)
 		)
-		(property "Part Number" "ERJ-2RKF1001X"
+		(property "Part Number" "RMCF0603FT1K00"
 			(at 200.66 118.11 90)
 			(effects
