File: modules/TC2030_PORTS.kicad_sch (KiCad schematic)
At the start: 4 parts, among them J3 TC2030, J4 TC2030

Commit message: Cambio de layout, correccion de pinout
Parts:
- removed C28: 100nF, Capacitor_SMD:C_0402_1005Metric, symbol Device:C
- renumbered C27 to C21
Other:
- moved on the sheet: C21, J3

Commit message: finishing version 1.0
Connections:
- net RP_SWO: no longer names the net of J3.6
- no-connect marks 0 -> 1
Changed lines of the file:
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@@
 	(paper "A4")
+	(junction
+		(at 176.53 78.74)
+		(diameter 0)
+		(color 0 0 0 0)
+	)
 	(junction
 		(at 85.09 78.74)
@@
 		(color 0 0 0 0)
 	)
+	(junction
+		(at 92.71 78.74)
+		(diameter 0)
+		(color 0 0 0 0)
+	)
+	(no_connect
+		(at 116.84 102.87)
+	)
 	(wire
 		(pts
@@
 	(wire
 		(pts
-			(xy 116.84 102.87) (xy 121.92 102.87)
-		)
-		(stroke
-			(width 0)
-			(type default)
-		)
-	)
-	(wire
-		(pts
 			(xy 104.14 102.87) (xy 99.06 102.87)
 		)
@@
 	(wire
 		(pts
-			(xy 168.91 78.74) (xy 189.23 78.74)
+			(xy 168.91 78.74) (xy 176.53 78.74)
 		)
 		(stroke
@@
 	(wire
 		(pts
+			(xy 92.71 78.74) (xy 105.41 78.74)
+		)
+		(stroke
+			(width 0)
+			(type default)
+		)
+	)
+	(wire
+		(pts
 			(xy 85.09 97.79) (xy 104.14 97.79)
 		)
@@
 	(wire
 		(pts
-			(xy 85.09 78.74) (xy 105.41 78.74)
+			(xy 85.09 78.74) (xy 92.71 78.74)
 		)
 		(stroke
@@
 		(pts
 			(xy 99.06 102.87) (xy 99.06 106.68)
+		)
+		(stroke
+			(width 0)
+			(type default)
+		)
+	)
+	(wire
+		(pts
+			(xy 176.53 78.74) (xy 189.23 78.74)
 		)
 		(stroke
@@
 		(shape bidirectional)
 		(at 121.92 97.79 0)
-		(effects
-			(font
-				(size 1.27 1.27)
-			)
-			(justify left)
-		)
-	)
-	(hierarchical_label "RP_SWO"
-		(shape output)
-		(at 121.92 102.87 0)
 		(effects
 			(font
@@
 	)
 	(symbol
+		(lib_id "power:PWR_FLAG")
+		(at 92.71 78.74 0)
+		(unit 1)
+		(exclude_from_sim no)
+		(in_bom yes)
+		(on_board yes)
+		(dnp no)
+		(fields_autoplaced yes)
+		(property "Reference" "#FLG04"
+			(at 92.71 76.835 0)
+			(effects
+				(font
+					(size 1.27 1.27)
+				)
+				(hide yes)
+			)
+		)
+		(property "Value" "PWR_FLAG"
+			(at 92.71 73.66 0)
+			(effects
+				(font
+					(size 1.27 1.27)
+				)
+			)
+		)
+		(property "Footprint" ""
+			(at 92.71 78.74 0)
+			(effects
+				(font
+					(size 1.27 1.27)
+				)
+				(hide yes)
+			)
+		)
+		(property "Datasheet" "~"
+			(at 92.71 78.74 0)
+			(effects
+				(font
+					(size 1.27 1.27)
+				)
+				(hide yes)
+			)
+		)
+		(property "Description" "Special symbol for telling ERC where power comes from"
+			(at 92.71 78.74 0)
+			(effects
+				(font
+					(size 1.27 1.27)
+				)
+				(hide yes)
+			)
+		)
+		(pin "1"
+		)
+		(instances
+			(project "RP_devBoard"
+				(path "/3efb3214-cf20-4475-a403-c426a77bfef6/f94e9cec-54f7-45dd-9630-aa4b6ec1eb86"
+					(reference "#FLG04")
+					(unit 1)
+				)
+			)
+		)
+	)
+	(symbol
 		(lib_id "power:GND")
 		(at 222.25 105.41 0)
@@
 					(unit 1)
 				)
+			)
+		)
+	)
+	(symbol
+		(lib_id "power:PWR_FLAG")
+		(at 176.53 78.74 0)
+		(unit 1)
+		(exclude_from_sim no)
+		(in_bom yes)
+		(on_board yes)
+		(dnp no)
+		(fields_autoplaced yes)
+		(property "Reference" "#FLG05"
+			(at 176.53 76.835 0)
+			(effects
+				(font
+					(size 1.27 1.27)
+				)
+				(hide yes)
+			)
+		)
+		(property "Value" "PWR_FLAG"
+			(at 176.53 73.66 0)
+			(effects
+				(font
+					(size 1.27 1.27)
+				)
+			)
+		)
+		(property "Footprint" ""
+			(at 176.53 78.74 0)
+			(effects
+				(font
+					(size 1.27 1.27)
+				)
+				(hide yes)
+			)
+		)
+		(property "Datasheet" "~"
+			(at 176.53 78.74 0)
+			(effects
+				(font
+					(size 1.27 1.27)
+				)
+				(hide yes)
+			)
+		)
+		(property "Description" "Special symbol for telling ERC where power comes from"
+			(at 176.53 78.74 0)
+			(effects
+				(font
+					(size 1.27 1.27)
+				)
+				(hide yes)
+			)
+		)
+		(pin "1"
+		)
+		(instances
+			(project "RP_devBoard"
+				(path "/3efb3214-cf20-4475-a403-c426a77bfef6/f94e9cec-54f7-45dd-9630-aa4b6ec1eb86"
+					(reference "#FLG05")
+					(unit 1)
+				)
