File: RP_devBoard.kicad_pcb (KiCad board)
At the start: 4 copper layers, 100 x 60 mm, 117 parts, among them J1 Conn_01x04, J2 Conn_01x04, J3 TC2030, J4 TC2030, J5 Conn_02x08_Counter_Clockwise, J6 USB_C_Receptacle, J7 Conn_02x08_Counter_Clockwise, Q2 AO3400A, Q3 AO3401A, SW1 SW_Push, SW3 SW_Push, SW4 SW_Push, SW5 SW, U1 RP2350B, U10 USBLC6-2SC6, U12 BME280, U2 ESP32-C3-WROOM-02, U4 TPS628502, U5 W25Q128JVS, U7 MAX40200AUK, U8 MAX40200AUK, U9 MAX40200AUK, Y1 12MHz

Commit message: Cambio de layout, correccion de pinout
Parts:
- removed C22, C23, C27, C37: 100nF, Capacitor_SMD:C_0402_1005Metric
- removed R24: 1K, Resistor_SMD:R_0402_1005Metric
- removed R25: 10k, Resistor_SMD:R_0603_1608Metric
- removed TP10, TP11, TP6: TestPoint, TestPoint:TestPoint_THTPad_D1.0mm_Drill0.5mm
- removed the TP21 at (1.02, 1.02)
- removed the TP21 at (125.2, 93.2)
- removed the TP22 at (1.02, 4.08)
- removed the TP22 at (127.4, 93.2)
- removed the TP25 at (1.02, 7.12)
- removed the TP25 at (123.0, 93.2)
- added C21: 100nF, Capacitor_SMD:C_0402_1005Metric, F.Cu at (116.0, 72.0)
- added H1: MountingHole, MountingHole:MountingHole_3.2mm_M3, F.Cu at (204.0, 52.5)
- added H2: MountingHole, MountingHole:MountingHole_3.2mm_M3, F.Cu at (204.0, 107.5)
- added H3: MountingHole, MountingHole:MountingHole_3.2mm_M3, F.Cu at (96.0, 107.5)
- added H4: MountingHole, MountingHole:MountingHole_3.2mm_M3, F.Cu at (96.0, 52.5)
- added R21: 10k, Resistor_SMD:R_0603_1608Metric, F.Cu at (193.2, 60.4)
- added R5: 2.2K, Resistor_SMD:R_0603_1608Metric, F.Cu at (189.3, 108.9)
- added TP21: TestPoint, Sadman_TP:TP_2.8mm_1mm, B.Cu at (157.9, 74.6)
- added TP22: TestPoint, Sadman_TP:TP_2.8mm_1mm, B.Cu at (153.9, 67.0)
- added TP25: TestPoint, Sadman_TP:TP_2.8mm_1mm, B.Cu at (161.9, 74.5)
- added TP26: TestPoint, Sadman_TP:TP_2.8mm_1mm, B.Cu at (155.7, 82.5)
- added TP27: TestPoint, Sadman_TP:TP_2.8mm_1mm, B.Cu at (176.0, 82.5)
- added TP28: TestPoint, Sadman_TP:TP_2.8mm_1mm, B.Cu at (172.0, 82.5)
- added TP29: TestPoint, Sadman_TP:TP_2.8mm_1mm, B.Cu at (168.0, 82.5)
- added TP30: TestPoint, Sadman_TP:TP_2.8mm_1mm, B.Cu at (163.9, 82.5)
- added TP31: TestPoint, Sadman_TP:TP_2.8mm_1mm, B.Cu at (151.6, 82.5)
- added TP32: TestPoint, Sadman_TP:TP_2.8mm_1mm, B.Cu at (147.5, 82.5)
- added TP33: TestPoint, Sadman_TP:TP_2.8mm_1mm, B.Cu at (143.5, 82.5)
- C16, C38, C8, C9: footprint Capacitor_SMD:C_0402_1005Metric -> Capacitor_SMD:C_0603_1608Metric
- C18: value 15pF -> 100nF; footprint Capacitor_SMD:C_0402_1005Metric -> Capacitor_SMD:C_0603_1608Metric
- C19: value 15pF -> 100nF
- C25: value 100nF -> 10uF; footprint Capacitor_SMD:C_0402_1005Metric -> Capacitor_SMD:C_0603_1608Metric
- C36: value 10uF -> 100nF
- C5: value 100nF -> 15pF
- C6: value 4.7uF -> 15pF; footprint Capacitor_SMD:C_0603_1608Metric -> Capacitor_SMD:C_0402_1005Metric
- C7: value 100nF -> 4.7uF
- R18: value 2.2K -> 1K
- R20: value 10k -> 1K; footprint Resistor_SMD:R_0603_1608Metric -> Capacitor_SMD:C_0603_1608Metric
- R6: footprint Resistor_SMD:R_0402_1005Metric -> Resistor_SMD:R_0603_1608Metric
- R8: value 1K -> 10k; footprint Resistor_SMD:R_0402_1005Metric -> Resistor_SMD:R_0603_1608Metric
- TP1: footprint Connector_Pin:Pin_D1.0mm_L10.0mm -> Sadman_TP:TP_2.8mm_1mm
- TP12, TP13, TP14, TP15, TP16, TP17, TP18, TP23, TP24, TP3, TP7, TP8, TP9: footprint TestPoint:TestPoint_THTPad_D1.0mm_Drill0.5mm -> Sadman_TP:TP_2.8mm_1mm
- TP19, TP20: footprint TestPoint:TestPoint_Pad_D1.0mm -> Sadman_TP:TP_2.8mm_1mm
- TP2: footprint Connector_Pin:Pin_D1.0mm_L10.0mm -> Sadman_TP:TP_2.8mm_1mm; moved to B.Cu
- TP4: footprint TestPoint:TestPoint_THTPad_D1.0mm_Drill0.5mm -> Sadman_TP:TP_2.8mm_1mm; moved to F.Cu
- TP5: footprint TestPoint:TestPoint_THTPad_D1.5mm_Drill0.7mm -> Sadman_TP:TP_2.8mm_1mm
- moved C25 276.0 mm to (199.1, 60.5), turned to 180 degrees
- moved R13 262.3 mm to (189.2, 60.4), turned to 180 degrees
- moved R23 258.0 mm to (184.8, 65.0), turned to 180 degrees
- moved R20 189.5 mm to (137.4, 53.5)
- moved R19 183.1 mm to (143.4, 56.5), turned to 90 degrees
- moved SW4 180.5 mm to (142.4, 52.5)
- moved R8 177.7 mm to (132.7, 56.4), turned to 90 degrees
- moved SW3 176.1 mm to (130.9, 52.5)
- moved C31 149.2 mm to (142.0, 74.9), turned to -90 degrees
- moved C32 143.5 mm to (134.5, 73.9), turned to 180 degrees
- moved BZ1 89.1 mm to (170.7, 54.6), turned to 90 degrees
- moved TP17 83.7 mm to (159.7, 82.5), turned to 90 degrees
- moved Q2 82.1 mm to (175.4, 62.5), turned to 0 degrees
- moved D2 77.2 mm to (170.5, 60.6), turned to 0 degrees
- moved C28 76.4 mm to (133.0, 66.4), turned to 90 degrees
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- renumbered J5 to J2, J7 to J5, J2 to J7, Q3 to Q1, R21 to R10, R12 to R11, R4 to R12, R5 to R17, R17 to R4, R11 to R9, SW5 to SW2, U10 to U3, U12 to U6
Connections:
- net Net-(U1-VREG_AVDD) renamed /RP2350B/VGREX_AVDD
- C10 pad 1: +3V3 -> +1V1
- C11 pad 1: +3V3 -> +1V1
- C12 pad 1: +3V3 -> +1V1
- C16 pad 1: +3V3 -> Net-(U1-GPIO15)
- C18 pad 1: Net-(U1-XIN) -> Net-(U1-GPIO14)
- C19 pad 1: Net-(C19-Pad1) -> +3V3
- C24 pad 1: +3V3 -> /ESP_EN
- C25 pad 1: /ESP_EN -> +3V3
- C28 pad 1: GND -> +3V3
- C28 pad 2: +3V3_TC2 -> GND
- C31 pad 1: Net-(U1-GPIO12) -> +3V3
- C32 pad 1: Net-(U1-GPIO11) -> +3V3
- C35 pad 1: /RP_NRESET -> +3V3
- C38 pad 1: +1V1 -> +3V3
- C4 pad 1: +3V3 -> +1V1
- C5 pad 1: +1V1 -> /RP2350B/RP_XIN
- C6 pad 1: +1V1 -> Net-(C6-Pad1)
- C8 pad 1: +1V1 -> +3V3
- C9 pad 1: +3V3 -> /RP_NRESET
- J2 pad 3: /RP_SS1 -> /RP_SS0
- J2 pad 5: /RP_MOSI -> /RP_MISO
- J2 pad 6: /RP_MISO -> /RP_MOSI
- J5 pad 1: /MK_AIN -> /MK_AIN2
- J5 pad 13: /MK_TX -> /MK_TX2
- J5 pad 14: /MK_RX -> /MK_RX2
- J5 pad 15: /MK_INT -> /MK_INT2
- J5 pad 16: /MK_PWM -> /MK_PWM2
- J5 pad 2: /MK_RST -> /MK_RST2
- J5 pad 3: /RP_SS2 -> /RP_SS1
- J5 pad 5: /RP_MOSI -> /RP_MISO
- J5 pad 6: /RP_MISO -> /RP_MOSI
- R13 pad 1: /ESP_EN -> Net-(U2-IO8)
- R18 pad 1: /SDA -> Net-(R18-Pad1)
- R19 pad 2: Net-(U1-GPIO12) -> Net-(U1-GPIO14)
- R20 pad 1: GND -> +3V3
- R20 pad 2: Net-(U1-GPIO11) -> Net-(R20-Pad2)
- R23 pad 1: Net-(U2-IO8) -> /ESP_BOOT
- R6 pad 1: Net-(C19-Pad1) -> GND
- R6 pad 2: Net-(U1-XOUT) -> Net-(R6-Pad2)
- R7 pad 1: GND -> Net-(C6-Pad1)
- R7 pad 2: Net-(R7-Pad2) -> /RP2350B/RP_XOUT
- R8 pad 1: Net-(R8-Pad1) -> GND
- R8 pad 2: Net-(U1-GPIO11) -> Net-(U1-GPIO15)
- SW1 pad 1: Net-(R7-Pad2) -> Net-(R6-Pad2)
- SW3 pad 1: Net-(U1-GPIO12) -> Net-(U1-GPIO15)
- SW3 pad 2: Net-(R24-Pad1) -> Net-(R18-Pad1)
- SW4 pad 1: Net-(R8-Pad1) -> Net-(U1-GPIO14)
- SW4 pad 2: +3V3 -> Net-(R20-Pad2)
- TP1 pad 1: GND -> VUSB0
- TP12 pad 1: /MK_AIN -> /MK_RST
- TP13 pad 1: /MK_RST -> /RP_SS0
- TP14 pad 1: /RP_SS1 -> /RP_CLK
- TP15 pad 1: /RP_CLK -> /RP_MOSI
- TP16 pad 1: /RP_MOSI -> /RP_MISO
- TP17 pad 1: /RP_MISO -> /MK_AIN2
- TP19 pad 1: Net-(U1-XIN) -> /MK_PWM
- TP2 pad 1: VUSB0 -> /USB0_DN
- TP20 pad 1: Net-(C19-Pad1) -> /MK_INT
- TP3 pad 1: +5V -> GND
- TP7 pad 1: /USB0_DP -> +5V
- TP8 pad 1: /USB0_DN -> /USB0_DP
- TP9 pad 1: +3V3_USB -> /MK_AIN
- U1 pad 1: /MK_RX -> /RP_SS2
- U1 pad 11: Net-(U1-GPIO12) -> unconnected-(U1-GPIO12-Pad11)
- U1 pad 13: unconnected-(U1-GPIO14-Pad13) -> Net-(U1-GPIO14)
- U1 pad 14: unconnected-(U1-GPIO15-Pad14) -> Net-(U1-GPIO15)
- U1 pad 2: /MK_TX -> unconnected-(U1-GPIO5-Pad2)
- U1 pad 23: /RP_SWO -> unconnected-(U1-GPIO23-Pad23)
- U1 pad 25: /BZZ_PWM -> unconnected-(U1-GPIO24-Pad25)
- U1 pad 3: /MK_PWM -> unconnected-(U1-GPIO6-Pad3)
- U1 pad 30: Net-(U1-XIN) -> /RP2350B/RP_XIN
- U1 pad 31: Net-(U1-XOUT) -> /RP2350B/RP_XOUT
- U1 pad 36: unconnected-(U1-GPIO28-Pad36) -> /RP_MOSI
- U1 pad 37: unconnected-(U1-GPIO29-Pad37) -> /RP_MISO
- U1 pad 38: unconnected-(U1-GPIO30-Pad38) -> /RP_CLK
- U1 pad 39: unconnected-(U1-GPIO31-Pad39) -> /RP_SS0
- U1 pad 4: /MK_INT -> unconnected-(U1-GPIO7-Pad4)
- U1 pad 42: unconnected-(U1-GPIO33-Pad42) -> /MK_PWM
- U1 pad 43: /RP_SS2 -> /MK_INT
- U1 pad 44: /RP_MISO -> /RP_SS1
- U1 pad 45: /RP_MOSI -> /MK_RX
- U1 pad 46: /RP_CLK -> /MK_TX
- U1 pad 47: /RP_SS0 -> /MK_RST2
- U1 pad 48: /RP_SS1 -> unconnected-(U1-GPIO39-Pad48)
- U1 pad 53: unconnected-(U1-GPIO40_ADC2-Pad53) -> /MK_RST
- U1 pad 54: unconnected-(U1-GPIO40_ADC3-Pad54) -> /MK_AIN2
- U1 pad 55: unconnected-(U1-GPIO40_ADC4-Pad55) -> /MK_PWM2
- U1 pad 56: unconnected-(U1-GPIO40_ADC5-Pad56) -> /MK_INT2
- U1 pad 57: unconnected-(U1-GPIO40_ADC6-Pad57) -> /MK_RX2
- U1 pad 58: unconnected-(U1-GPIO40_ADC7-Pad58) -> /MK_TX2
- U1 pad 6: /MK_RST -> unconnected-(U1-GPIO8-Pad6)
- U1 pad 80: unconnected-(U1-GPIO3-Pad80) -> /BZZ_PWM
- U1 pad 9: Net-(U1-GPIO11) -> unconnected-(U1-GPIO11-Pad9)
- U2 pad 10: /RP_SS0 -> /RP_SS2
- Y1 pad 1: Net-(C19-Pad1) -> Net-(C6-Pad1)
- Y1 pad 3: Net-(U1-XIN) -> /RP2350B/RP_XIN
Routing:
- net /MK_TX2: track 0.00 -> 62.4 mm, vias 0 -> 2
- net /RP_MISO: track 91.3 -> 149.4 mm, vias 2 -> 4
- net /RP_SS2: track 0.00 -> 57.0 mm, vias 0 -> 4
- net /MK_RX2: track 0.00 -> 55.9 mm, vias 0 -> 2
- net /RP_MOSI: track 109.8 -> 164.5 mm, vias 2 -> 4
- net /MK_INT2: track 0.00 -> 49.0 mm
- net /MK_RST: track 4.08 -> 50.3 mm, vias 0 -> 2
- net /MK_TX: track 0.00 -> 46.2 mm, vias 0 -> 1
- net /ESP_BOOT: track 0.00 -> 45.6 mm, vias 0 -> 2
- net /RP_NRESET: track 7.56 -> 52.8 mm, vias 0 -> 2
- net /MK_AIN2: track 0.00 -> 43.9 mm
- net /MK_PWM2: track 0.00 -> 43.0 mm
- net /MK_RST2: track 0.00 -> 42.6 mm, vias 0 -> 1
- net /RP_SS0: track 0.00 -> 37.2 mm, vias 0 -> 1
- net /MK_RX: track 0.00 -> 36.8 mm, vias 0 -> 1
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- added copper zone on In2.Cu, net +1V1
- added copper zone on In2.Cu, net +3V3
- added copper zone on In2.Cu, net +3V3_USB
- added copper zone on In2.Cu, net +5V
- added copper zone on F.Cu, net /POWER/SW_SOURCE
- added copper zone on B.Cu, net GND
- added copper zone on F.Cu, net GND
- added copper zone on In1.Cu, net GND
- added copper zone on In2.Cu, net GND
- added copper zone on In2.Cu, net VUSB0
Other:
- board size 100 x 60 mm -> 115 x 62 mm

Commit message: finishing version 1.0
Parts:
- H1, H2, H3, H4: footprint MountingHole:MountingHole_3.2mm_M3 -> MountingHole:MountingHole_3.2mm_M3_DIN965_Pad
- R20: footprint Capacitor_SMD:C_0603_1608Metric -> Resistor_SMD:R_0603_1608Metric
- TP1, TP19, TP20, TP4, TP5: moved to B.Cu
- moved C7 11.4 mm to (151.2, 75.4)
- moved C11 8.84 mm to (139.8, 74.9), turned to -90 degrees
- moved R20 5.84 mm to (143.2, 53.5)
- moved SW4 5.84 mm to (148.2, 52.5)
- moved TP5 0.52 mm to (152.3, 72.7), turned to 180 degrees
- moved TP18 0.51 mm to (163.3, 61.0)
- moved TP24 0.36 mm to (155.8, 60.9)
- moved TP23 0.24 mm to (159.6, 60.8)
- moved C8 0.18 mm to (147.5, 70.9)
- moved C39 0.14 mm to (138.5, 74.9)
- turned TP19 to 180 degrees
- turned TP20 to 180 degrees
- turned TP4 to 180 degrees
Connections:
- J3 pad 6: /RP_SWO -> unconnected-(J3-Pad6)
Routing:
- net /ESP_EN: track 8.03 -> 70.9 mm, vias 0 -> 4
- net Net-(Q1-G): track 7.57 -> 28.6 mm, vias 0 -> 2
- net /ESP_TX: track 25.8 -> 15.4 mm
- net /ESP_RX: track 29.3 -> 22.9 mm, vias 0 -> 2
- net Net-(U1-GPIO14): track 33.1 -> 38.3 mm
- net GND: track 62.6 -> 66.9 mm, vias 94 -> 101
- net +3V3: track 64.2 -> 67.3 mm, vias 43 -> 49
- net /ESP_BOOT: track 45.6 -> 46.4 mm
Other:
- board text added: "0"
- board text added: "0 mm"
- board text added: "0.0000 mm / 0.0000 mm"
- board text added: "0.01 mm"
- board text added: "0.02"
- board text added: "0.035 mm"
- board text added: "0.1 mm"
- board text added: "0.2000 mm"
- board text added: "1"
- board text added: "1.24 mm"
- board text added: "1.6000 mm"
- board text added: "115.0000 mm x 62.0000 mm"
- board text added: "3.3"
- board text added: "4"
- board text added: "4.5"
- board text added: "90 OHMS"
- board text added: "B.Cu"
- board text added: "B.Mask"
- board text added: "B.Paste"
- board text added: "B.Silkscreen"
- board text added: "BOARD CHARACTERISTICS"
- board text added: "Board Thickness:"
- board text added: "Board overall dimensions:"
- board text added: "Bottom Silk Screen"
- board text added: "Bottom Solder Mask"
- board text added: "Bottom Solder Paste"
- board text added: "Castellated pads:"
- board text added: "Color"
- board text added: "Copper Finish:"
- board text added: "Copper Layer Count:"
- board text added: "Dielectric 1"
- board text added: "Dielectric 2"
- board text added: "Dielectric 3"
- board text added: "Direct Printing"
- board text added: "Edge card connectors:"
- board text added: "Epsilon R"
- board text added: "F.Cu"
- board text added: "F.Mask"
- board text added: "F.Paste"
- board text added: "F.Silkscreen"
- board text added: "FR4"
- board text added: "FR4 natural"
- board text added: "Green"
- board text added: "Impedance Control:"
- board text added: "In1.Cu"
- board text added: "In2.Cu"
- board text added: "Layer Name"
- board text added: "Liquid Ink"
- board text added: "Loss Tangent"
- board text added: "Material"
- board text added: "Min hole diameter:"
- board text added: "Min track/spacing:"
- board text added: "No"
- board text added: "None"
- board text added: "Plated Board Edge:"
- board text added: "Thickness (mm)"
- board text added: "Top Silk Screen"
- board text added: "Top Solder Mask"
- board text added: "Top Solder Paste"
- board text added: "Type"
- board text added: "White"
- board text added: "Yes"
- board text added: "copper"
- board text added: "core"
- board text added: "prepreg"
